File: resources_for_zebra_fish/board/from_eagle/test1/test1.sch (KiCad schematic (older format))
At the start: 25 parts, among them J1 enable, M1 30V, M2 30V, U1 LM3150MH/NOPB

Commit message: completed lm3150 pcb
Connections:
- wire segments 68 -> 69
Changed lines of the file:
@@
 	10750 4800 10800 4800
 Wire Wire Line
-	10000 4800 10800 4800
+	10000 4800 10750 4800
 Wire Wire Line
 	2900 4950 3850 4950
@@
 Wire Wire Line
 	3850 4400 4200 4400
+Connection ~ 10750 4800
+Wire Wire Line
+	10750 4800 10800 4800
 $EndSCHEMATC
