File: resources_for_zebra_fish/boards/Lcr_addon/Lcr_addon.kicad_pcb (KiCad board)
At the start: 2 copper layers, 85.1 x 59.9 mm, 26 parts, among them J1 12V_in, J2 LCr_ conector, J3 power source, J4 blank in, J5 Green control output, J6 Blue control output, J7 Red control output, J8 blank_jumper, U1 RED channel, U2 Green channel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

Commit message: update LCr board
Parts:
- removed J1: 12V_in, Connector_BarrelJack:BarrelJack_Horizontal
- removed J3: power source, Connector_PinHeader_2.54mm:PinHeader_1x03_P2.54mm_Vertical
- removed R2, R3: 1k, Resistor_THT:R_Axial_DIN0207_L6.3mm_D2.5mm_P10.16mm_Horizontal
- removed the REF** at (42.2, 56.9)
- removed the REF** at (116.3, 56.9)
- removed the REF** at (116.3, 106.2)
- added REF**: MountingHole_3.2mm_M3_ISO14580_Pad, MountingHole:MountingHole_3.2mm_M3_ISO14580_Pad, F.Cu at (116.8, 56.4)
- added REF**: MountingHole_3.2mm_M3_ISO14580_Pad, MountingHole:MountingHole_3.2mm_M3_ISO14580_Pad, F.Cu at (114.3, 56.4)
- added REF**: MountingHole_3.2mm_M3_ISO14580_Pad, MountingHole:MountingHole_3.2mm_M3_ISO14580_Pad, F.Cu at (43.7, 56.4)
- added REF**: MountingHole_3.2mm_M3_ISO14580_Pad, MountingHole:MountingHole_3.2mm_M3_ISO14580_Pad, F.Cu at (41.1, 56.4)
- R1: footprint Resistor_THT:R_Axial_DIN0207_L6.3mm_D2.5mm_P10.16mm_Horizontal -> Resistor_THT:R_Axial_DIN0207_L6.3mm_D2.5mm_P2.54mm_Vertical
- U8: value TC7S14F -> 74AHC1G04
- moved J8 16.3 mm to (116.3, 72.1)
- moved U8 9.91 mm to (75.2, 76.7)
- moved J4 6.83 mm to (108.2, 93.5)
- moved J6 5.92 mm to (86.9, 93.5)
- moved J5 5.30 mm to (68.6, 93.5)
- moved U2 5.09 mm to (54.4, 71.6)
- moved U3 5.09 mm to (54.4, 61.5)
- moved U7 5.09 mm to (61.5, 61.5)
- moved J7 5.08 mm to (50.3, 93.5)
- moved U6 5.08 mm to (61.5, 71.6)
- moved U1 4.83 mm to (54.4, 81.8)
- moved U5 4.83 mm to (62.0, 81.8)
- moved R1 0.52 mm to (90.4, 79.2)
Connections:
- C1 pad 1: Net-(C1-Pad1) -> +12V
- J2 pad 1: Net-(J2-Pad1) -> +12V
- R1 pad 1: GND -> Net-(J4-Pad1)
- R1 pad 2: Net-(J7-Pad1) -> Net-(R1-Pad2)
- U4 pad 1: Net-(C1-Pad1) -> +12V
- U8 pad 1: Net-(U8-Pad1) -> (no net)
- U8 pad 2: Net-(J4-Pad1) -> Net-(R1-Pad2)
Routing:
- net Net-(J2-Pad1): track 49.6 -> 0.00 mm
- net Net-(C1-Pad1): track 22.9 -> 0.00 mm
- net Net-(J7-Pad1): track 44.9 -> 22.3 mm, vias 2 -> 0
- net Net-(J5-Pad1): track 47.7 -> 25.6 mm, vias 1 -> 0
- net +12V: track 54.2 -> 72.6 mm
- net Net-(R1-Pad2): track 0.00 -> 15.1 mm, vias 0 -> 1
- net Net-(J4-Pad1): track 39.9 -> 27.5 mm
- net Net-(J8-Pad2): track 89.7 -> 77.7 mm
- net Net-(J2-Pad9): track 13.7 -> 23.7 mm, vias 0 -> 1
- net Net-(J6-Pad1): track 56.6 -> 47.4 mm, vias 3 -> 2
- net VCC: track 157.2 -> 148.2 mm, vias 7 -> 4
- net Net-(J2-Pad8): track 19.8 -> 13.0 mm, vias 3 -> 1
- net Net-(U3-Pad4): track 11.7 -> 6.58 mm
- net Net-(J8-Pad1): track 39.3 -> 44.2 mm
- net Net-(J2-Pad10): track 11.9 -> 14.7 mm
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Other:
- board size 85.1 x 59.9 mm -> 85.1 x 55.1 mm

Commit message: clean up add on board
Parts:
- U8: value 74AHC1G04 -> Signal Inverter
Changed lines of the file:
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@@
       (effects (font (size 1 1) (thickness 0.15)))
     )
-    (fp_text value 74AHC1G04 (at 0 2.5 90) (layer F.SilkS)
+    (fp_text value "Signal Inverter" (at 0 2.5 90) (layer F.SilkS)
       (effects (font (size 1 1) (thickness 0.15)))
     )
@@
   (segment (start 94.488 54.72) (end 103.408 54.72) (width 0.25) (layer F.Cu) (net 2) (status 20))
   (segment (start 94.488 54.72) (end 94.488 54.74) (width 0.25) (layer F.Cu) (net 2))
-  (segment (start 81.534 68.326) (end 81.534 59.69) (width 0.25) (layer F.Cu) (net 3) (status 10))
-  (segment (start 89.943999 53.820001) (end 91.44 52.324) (width 0.25) (layer B.Cu) (net 3))
-  (segment (start 96.012 52.324) (end 103.632 59.944) (width 0.25) (layer B.Cu) (net 3) (status 20))
-  (segment (start 91.44 52.324) (end 96.012 52.324) (width 0.25) (layer B.Cu) (net 3))
-  (segment (start 87.696 55.372) (end 89.076 56.752) (width 0.25) (layer F.Cu) (net 3) (status 20))
-  (segment (start 81.534 59.69) (end 85.852 55.372) (width 0.25) (layer F.Cu) (net 3))
-  (segment (start 89.943999 53.820001) (end 89.435999 53.820001) (width 0.25) (layer B.Cu) (net 3))
-  (via (at 87.884 55.372) (size 0.8) (drill 0.4) (layers F.Cu B.Cu) (net 3))
-  (segment (start 89.435999 53.820001) (end 87.884 55.372) (width 0.25) (layer B.Cu) (net 3))
-  (segment (start 87.884 55.372) (end 86.868 55.372) (width 0.25) (layer F.Cu) (net 3))
-  (segment (start 85.852 55.372) (end 86.868 55.372) (width 0.25) (layer F.Cu) (net 3))
-  (segment (start 86.868 55.372) (end 87.696 55.372) (width 0.25) (layer F.Cu) (net 3))
-  (segment (start 87.376 57.524) (end 87.376 60.452) (width 0.25) (layer B.Cu) (net 4) (status 20))
-  (segment (start 78.994 55.372) (end 85.224 55.372) (width 0.25) (layer B.Cu) (net 4) (status 10))
-  (segment (start 85.224 55.372) (end 87.376 57.524) (width 0.25) (layer B.Cu) (net 4))
   (segment (start 105.41 74.456) (end 104.682 75.184) (width 0.25) (layer B.Cu) (net 2))
   (segment (start 105.41 73.406) (end 105.41 74.456) (width 0.25) (layer B.Cu) (net 2))
@@
   (segment (start 111.633 67.056) (end 116.332 67.056) (width 0.25) (layer F.Cu) (net 2))
   (segment (start 107.696 70.993) (end 111.633 67.056) (width 0.25) (layer F.Cu) (net 2))
+  (segment (start 81.534 68.326) (end 81.534 59.69) (width 0.25) (layer F.Cu) (net 3) (status 10))
+  (segment (start 89.943999 53.820001) (end 91.44 52.324) (width 0.25) (layer B.Cu) (net 3))
+  (segment (start 96.012 52.324) (end 103.632 59.944) (width 0.25) (layer B.Cu) (net 3) (status 20))
+  (segment (start 91.44 52.324) (end 96.012 52.324) (width 0.25) (layer B.Cu) (net 3))
+  (segment (start 87.696 55.372) (end 89.076 56.752) (width 0.25) (layer F.Cu) (net 3) (status 20))
+  (segment (start 81.534 59.69) (end 85.852 55.372) (width 0.25) (layer F.Cu) (net 3))
+  (segment (start 89.943999 53.820001) (end 89.435999 53.820001) (width 0.25) (layer B.Cu) (net 3))
+  (via (at 87.884 55.372) (size 0.8) (drill 0.4) (layers F.Cu B.Cu) (net 3))
+  (segment (start 89.435999 53.820001) (end 87.884 55.372) (width 0.25) (layer B.Cu) (net 3))
+  (segment (start 87.884 55.372) (end 86.868 55.372) (width 0.25) (layer F.Cu) (net 3))
+  (segment (start 85.852 55.372) (end 86.868 55.372) (width 0.25) (layer F.Cu) (net 3))
+  (segment (start 86.868 55.372) (end 87.696 55.372) (width 0.25) (layer F.Cu) (net 3))
+  (segment (start 87.376 57.524) (end 87.376 60.452) (width 0.25) (layer B.Cu) (net 4) (status 20))
+  (segment (start 78.994 55.372) (end 85.224 55.372) (width 0.25) (layer B.Cu) (net 4) (status 10))
+  (segment (start 85.224 55.372) (end 87.376 57.524) (width 0.25) (layer B.Cu) (net 4))
   (segment (start 41.91 80.518) (end 43.18 80.518) (width 0.25) (layer B.Cu) (net 4))
   (segment (start 69.596 55.372) (end 69.088 54.864) (width 0.25) (layer B.Cu) (net 4))
@@
     (connect_pads (clearance 0.508))
     (min_thickness 0.254)
-    (fill yes (arc_segments 16) (thermal_gap 0.508) (thermal_bridge_width 0.508))
+    (fill (arc_segments 16) (thermal_gap 0.508) (thermal_bridge_width 0.508))
     (polygon
       (pts
