File: boards/mosfet_circuit/led_driver.kicad_pcb (KiCad board)
At the start: 2 copper layers, 67.3 x 33 mm, 11 parts, among them J1 Vin, J2 control_in, J4 LED, Q1 N_chan_mosfet, Q2 P-Chan_mosfet

Commit message: preparing boards for kitspace
Other:
- board text added: "1"
Changed lines of the file:
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@@
   (general
     (thickness 1.6)
-    (drawings 9)
+    (drawings 11)
     (tracks 42)
     (zones 0)
@@
     (pad 1 np_thru_hole circle (at 0 0) (size 3.2 3.2) (drill 3.2) (layers *.Cu *.Mask))
   )
+  (gr_text 1 (at 179.9082 70.485) (layer F.SilkS)
+    (effects (font (size 1.5 1.5) (thickness 0.3)))
+  )
+  (gr_text 1 (at 189.5094 85.344) (layer F.SilkS)
+    (effects (font (size 1.5 1.5) (thickness 0.3)))
+  )
   (target plus (at 161.544 99.06) (size 5) (width 0.1) (layer Edge.Cuts))
