File: boards/mosfet_circuit_plus_voltage_regulator/led_driver.sch (KiCad schematic (older format))
At the start: 25 parts, among them J1 Vin, J2 LED, J3 control_in, Q1 N_chan_mosfet, Q2 P-Chan_mosfet, U1 MC34063AP

Commit message: final first draft of new board. now to order it and test
Parts:
- added H4: MountingHole, MountingHole:MountingHole_3.2mm_M3, symbol Mechanical:MountingHole
Changed lines of the file:
@@
+	1    0    0    -1
+$EndComp
+$Comp
+L Mechanical:MountingHole H4
+U 1 1 5D2610E5
+P 6150 2800
+F 0 "H4" H 6250 2846 50  0000 L CNN
+F 1 "MountingHole" H 6250 2755 50  0000 L CNN
+F 2 "MountingHole:MountingHole_3.2mm_M3" H 6150 2800 50  0001 C CNN
+F 3 "~" H 6150 2800 50  0001 C CNN
+	1    6150 2800
 	1    0    0    -1
 $EndComp

Commit message: fixed board foot prints
Parts:
- L1: footprint Inductor_THT:L_Radial_D7.0mm_P3.00mm -> Inductor_THT:L_Radial_D7.5mm_P5.00mm_Fastron_07P
- R2: footprint Resistor_THT:R_Axial_DIN0207_L6.3mm_D2.5mm_P10.16mm_Horizontal -> Resistor_THT:R_Axial_DIN0414_L11.9mm_D4.5mm_P15.24mm_Horizontal
- R7: footprint Resistor_THT:R_Axial_DIN0207_L6.3mm_D2.5mm_P10.16mm_Horizontal -> Package_TO_SOT_THT:TO-220-2_Vertical
- RV1: footprint Potentiometer_THT:Potentiometer_ACP_CA14-H5_Horizontal -> Potentiometer_THT:Potentiometer_Vishay_T73YP_Vertical
Changed lines of the file:
@@
 F 0 "R7" V 9243 3550 50  0000 C CNN
 F 1 "0.5 20W" V 9334 3550 50  0000 C CNN
-F 2 "Resistor_THT:R_Axial_DIN0207_L6.3mm_D2.5mm_P10.16mm_Horizontal" V 9380 3550 50  0001 C CNN
+F 2 "Package_TO_SOT_THT:TO-220-2_Vertical" V 9380 3550 50  0001 C CNN
 F 3 "~" H 9450 3550 50  0001 C CNN
 	1    9450 3550
@@
 F 0 "R2" V 1793 3100 50  0000 C CNN
 F 1 "0.22ohm" V 1884 3100 50  0000 C CNN
-F 2 "Resistor_THT:R_Axial_DIN0207_L6.3mm_D2.5mm_P10.16mm_Horizontal" V 1930 3100 50  0001 C CNN
+F 2 "Resistor_THT:R_Axial_DIN0414_L11.9mm_D4.5mm_P15.24mm_Horizontal" V 1930 3100 50  0001 C CNN
 F 3 "~" H 2000 3100 50  0001 C CNN
 	1    2000 3100
@@
 F 0 "RV1" V 3436 4250 50  0000 C CNN
 F 1 "5kohm" V 3345 4250 50  0000 C CNN
-F 2 "Potentiometer_THT:Potentiometer_ACP_CA14-H5_Horizontal" H 3550 4250 50  0001 C CNN
+F 2 "Potentiometer_THT:Potentiometer_Vishay_T73YP_Vertical" H 3550 4250 50  0001 C CNN
 F 3 "~" H 3550 4250 50  0001 C CNN
 	1    3550 4250
@@
 F 0 "L1" V 3750 3850 50  0000 C CNN
 F 1 "120µH" V 3850 3850 50  0000 C CNN
-F 2 "Inductor_THT:L_Radial_D7.0mm_P3.00mm" H 3900 3850 50  0001 C CNN
+F 2 "Inductor_THT:L_Radial_D7.5mm_P5.00mm_Fastron_07P" H 3900 3850 50  0001 C CNN
 F 3 "~" H 3900 3850 50  0001 C CNN
 	1    3900 3850
