File: boards/lcr_add-on/Lcr_addon.kicad_pcb (KiCad board)
At the start: 2 copper layers, 85.1 x 55.1 mm, 23 parts, among them J2 LCr_ conector, J4 blank in, J5 Green control output, J6 Blue control output, J7 Red control output, J8 blank_jumper, U1 RED channel, U2 Green channel, U3 Blue channel, U4 LM2596T-5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

Commit message: final wiring for lcr board
Parts:
- removed U5: RED+blank, Package_SO:TSOP-5_1.65x3.05mm_P0.95mm
- removed U6: Green+blank, Package_SO:TSOP-5_1.65x3.05mm_P0.95mm
- removed U7: Blue+blank, Package_SO:TSOP-5_1.65x3.05mm_P0.95mm
- removed U8: Signal Inverter, Package_SO:TSOP-5_1.65x3.05mm_P0.95mm
- U1: value RED channel -> SN74LS08N; footprint Package_SO:TSOP-5_1.65x3.05mm_P0.95mm -> Package_DIP:DIP-14_W7.62mm_Socket_LongPads
- U2: value Green channel -> SN74LS08N; footprint Package_SO:TSOP-5_1.65x3.05mm_P0.95mm -> Package_DIP:DIP-14_W7.62mm_Socket_LongPads
- U3: value Blue channel -> SN74HC14N; footprint Package_SO:TSOP-5_1.65x3.05mm_P0.95mm -> Package_DIP:DIP-14_W7.62mm_Socket_LongPads
- moved U3 43.9 mm to (92.0, 84.0)
- moved R1 26.7 mm to (116.5, 85.0), turned to 90 degrees
- moved U1 12.8 mm to (55.0, 69.0)
- moved U2 11.4 mm to (55.0, 83.0)
- moved C2 6.12 mm to (107.0, 67.5)
- moved J8 2.11 mm to (115.0, 70.5)
Connections:
- net Net-(J2-Pad5) renamed red_sig1
- net Net-(J2-Pad8) renamed red_sig2
- C2 pad 1: VCC -> +5V
- J2 pad 10: Net-(J2-Pad10) -> blue_sig2
- J2 pad 11: Net-(J2-Pad11) -> (no net)
- J2 pad 2: Net-(J2-Pad2) -> (no net)
- J2 pad 3: Net-(J2-Pad3) -> (no net)
- J2 pad 4: Net-(J2-Pad4) -> (no net)
- J2 pad 6: Net-(J2-Pad6) -> green_sig1
- J2 pad 7: Net-(J2-Pad7) -> blue_sig1
- J2 pad 9: Net-(J2-Pad9) -> green_sig2
- J8 pad 1: Net-(J8-Pad1) -> inverted_blank
- J8 pad 2: Net-(J8-Pad2) -> inv_blank-or-5V-input
- J8 pad 3: VCC -> +5V
- L1 pad 2: VCC -> +5V
- U1 pad 3: GND -> Net-(U1-Pad3)
- U1 pad 4: Net-(U1-Pad4) -> green_sig1
- U1 pad 5: VCC -> green_sig2
- U2 pad 1: Net-(J2-Pad6) -> Net-(U1-Pad3)
- U2 pad 2: Net-(J2-Pad9) -> inv_blank-or-5V-input
- U2 pad 3: GND -> Net-(J7-Pad1)
- U2 pad 4: Net-(U2-Pad4) -> Net-(U1-Pad6)
- U2 pad 5: VCC -> inv_blank-or-5V-input
- U3 pad 1: Net-(J2-Pad7) -> Net-(R1-Pad2)
- U3 pad 2: Net-(J2-Pad10) -> inverted_blank
- U3 pad 3: GND -> (no net)
- U3 pad 5: VCC -> (no net)
- U4 pad 4: VCC -> +5V
Routing:
- net VCC: track 148.2 -> 0.00 mm, vias 4 -> 0
- net +5V: track 0.00 -> 134.5 mm
- net Net-(J8-Pad2): track 77.7 -> 0.00 mm, vias 4 -> 0
- net inv_blank-or-5V-input: track 0.00 -> 71.9 mm, vias 0 -> 2
- net Net-(J8-Pad1): track 44.2 -> 0.00 mm
- net blue_sig1: track 0.00 -> 37.9 mm
- net green_sig2: track 0.00 -> 32.3 mm
- net Net-(U1-Pad6): track 0.00 -> 29.1 mm, vias 0 -> 1
- net inverted_blank: track 0.00 -> 27.0 mm
- net blue_sig2: track 0.00 -> 24.8 mm, vias 0 -> 2
- net Net-(J2-Pad7): track 23.9 -> 0.00 mm, vias 1 -> 0
- net Net-(J2-Pad9): track 23.7 -> 0.00 mm, vias 1 -> 0
- net green_sig1: track 0.00 -> 20.6 mm
- net Net-(U1-Pad3): track 0.00 -> 18.5 mm, vias 0 -> 1
- net Net-(J6-Pad1): track 47.4 -> 29.9 mm, vias 2 -> 0
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- added copper zone on B.Cu, net GND
- removed copper zone on F.Cu, net GND

Commit message: final update
Other:
- rule pad_to_mask_clearance: 0.051 -> 0
Changed lines of the file:
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@@
     (pad_size 1.524 1.524)
     (pad_drill 0.762)
-    (pad_to_mask_clearance 0.051)
-    (solder_mask_min_width 0.25)
+    (pad_to_mask_clearance 0)
     (aux_axis_origin 39.624 103.505)
     (visible_elements FFFFFF7F)
@@
       (effects (font (size 1 1) (thickness 0.15)))
     )
-    (pad 1 thru_hole roundrect (at 0 0 90) (size 1.2 1.2) (drill 0.75) (layers *.Cu *.Mask) (roundrect_rratio 0.208333)
+    (pad 1 thru_hole roundrect (at 0 0 90) (size 1.2 1.2) (drill 0.75) (layers *.Cu *.Mask) (roundrect_rratio 0.2083325)
       (net 3 +12V))
     (pad 3 thru_hole circle (at 2 0 90) (size 1.2 1.2) (drill 0.75) (layers *.Cu *.Mask))
